File: Keyboard0.kicad_sch (KiCad schematic)
At the start: 0 parts

Commit message: Schema1
Parts:
- added C1, C2, C3, C4: 0.1u, symbol Device:C
- added C5: 10u, symbol Device:C
- added C6, C7: 22p, symbol Device:C
- added C8: 1u, symbol Device:C_Small
- added F1: 500m, symbol Device:Polyfuse_Small
- added J1: AVR-ISP-6, symbol Connector:AVR-ISP-6
- added R1: 10k, symbol Device:R
- added R2: 10k, symbol Device:R_Small
- added R3, R4: 22, symbol Device:R
- added R5, R6: 5.1k, symbol Device:R
- added SW84: SW_SKQG, symbol local:SW_SKQG
- added U1: ATmega32U4-A, Package_QFP:TQFP-44_10x10mm_P0.8mm, symbol MCU_Microchip_ATmega:ATmega32U4-A
- added U2: PRTR5V0U2X, symbol random-keyboard-parts:PRTR5V0U2X
- added USB1: HRO-TYPE-C-31-M-12, symbol Type-C:HRO-TYPE-C-31-M-12
- added Y1: XTAL, symbol Device:Crystal_GND24_Small
Connections:
- new net: R4.1, U2.2 (IO1), USB1.8 (DP2)
- new net: R3.1, U2.3 (IO2), USB1.5 (DN2), USB1.6 (DP1), USB1.7 (DN1)
- new net: C8.1, U1.6 (UCAP)
- new net: R5.1, USB1.10 (CC2)
- new net: R6.1, USB1.4 (CC1)
- new net: R2.1, U1.33 (~{HWB}/PE2)
- new net +5V: C1.1, C2.1, C3.1, C4.1, C5.1, F1.2, J1.2 (VCC), R1.1, U1.14 (VCC), U1.2 (UVCC), U1.24 (AVCC), U1.34 (VCC), U1.44 (AVCC), U1.7 (VBUS)
- new net D+: R4.2, U1.4 (D+)
- new net D-: R3.2, U1.3 (D-)
- new net GND: C1.2, C2.2, C3.2, C4.2, C5.2, C6.2, C7.2, C8.2, J1.6 (GND), R2.2, R5.2, R6.2, SW84.2, U1.15 (GND), U1.23 (GND), U1.35 (GND), U1.43 (GND), U1.5 (UGND), U2.1 (GND), USB1.1 (GND), USB1.12 (GND), USB1.13 (SHIELD), Y1.2, Y1.4
- new net MISO: J1.1 (MISO), U1.11 (PB3)
- new net MOSI: J1.4 (MOSI), U1.10 (PB2)
- new net RESET: J1.5 (~{RST}), R1.2, SW84.1, U1.13 (~{RESET})
- new net SCK: J1.3 (SCK), U1.9 (PB1)
- new net VCC: F1.1, U2.4 (VCC), USB1.11 (VBUS), USB1.2 (VBUS)
- new net XTAL1: C6.1, U1.17 (XTAL1), Y1.1
- new net XTAL2: C7.1, U1.16 (XTAL2), Y1.3
- no-connect marks 0 -> 5
Other:
- added sheet Matrix (matrix.kicad_sch)
